Commit message: working with ros2

File: description/urdf/Cart.urdf (robot description, URDF)
Before this commit: robot Cart, 2 links, 1 joints
Links:
- link Body: mass 10.0 -> 100.0

Commit message: testing

File: description/urdf/Cart.urdf (robot description, URDF)
Before this commit: robot Cart, 2 links, 1 joints
Links:
- link Body: mass 100.0 -> 1000.0

Commit message: reset mass to default

File: description/urdf/Cart.urdf (robot description, URDF)
Before this commit: robot Cart, 2 links, 1 joints
Links:
- link Body: mass 1000.0 -> 10.0
